Commit message: Fixed world frame in moveit config

File: src/saif_devices/src/robot_description/ur10_dual_arms.urdf (robot description, URDF)
Before this commit: robot ur10_two_arms, 24 links, 23 joints
Links:
- removed link world
- link platform: geometry visual box size=5.0 3.0 0.05
Joints:
- removed joint world_joint
- joint left_platform_base: origin xyz=-0.5 -0.5 0.0 rpy=0 0 0 -> xyz=-0.75 0 0.0 rpy=0 0 0
- joint right_platform_base: origin xyz=0.20 0.20 0.0 rpy=0 0 0 -> xyz=0.75 0.00 0.0 rpy=0 0 0
