Commit message: Added force torque sensor to moveit and urdf

File: src/saif_devices/src/dual_arm_description/urdf/blue.urdf.xacro (robot description, xacro)
@@ -4,8 +4,12 @@
 	<xacro:include filename="$(find ur_description)/urdf/common.gazebo.xacro" />
 	<xacro:include filename="$(find ur_description)/urdf/ur10.urdf.xacro" />
+	<xacro:include filename="$(find robotiq_ft_sensor)/urdf/robotiq_ft300.urdf.xacro"/>
+	<xacro:robotiq_ft300 parent="blue_tool0" prefix="blue_">
+		<origin xyz="0 0 0" rpy="0 0 0"/>
+	</xacro:robotiq_ft300>
 	<!-- arm -->
 	<xacro:ur10_robot prefix="blue_" joint_limited="false"/>
- 	<xacro:robotiq_85_gripper prefix="" parent="blue_ee_link">
-		 <origin xyz="0.0 0.0 0.0" rpy="0 0 0"/>
+ 	<xacro:robotiq_85_gripper prefix="" parent="blue_robotiq_ft_frame_id">
+		 <origin xyz="0.0 0.0 0.0" rpy="0 -1.57079632679 0"/>
 	</xacro:robotiq_85_gripper>
 </robot>
