Commit message: Fixed urdf 3 finger hand orientation, played with relative arm calibration, needs proper scheme

File: src/saif_devices/src/dual_arm_description/urdf/dual.urdf (robot description, URDF)
Before this commit: robot dual, 47 links, 46 joints
Joints:
- joint ceiling_to_blue: origin xyz=-0.75 0 0 -> xyz=-0.715 0.05 0
- joint ceiling_to_red: origin xyz=0.75 0 0 -> xyz=0.715 0 0
- joint red_palm_arm: origin xyz=0 0 0 rpy=1.57079632679 0 0 -> xyz=0 0 0 rpy=1.57079632679 0 2.35619449019

File: src/saif_devices/src/dual_arm_description/urdf/dual.urdf.xacro (robot description, xacro)
@@ -22,5 +22,5 @@
 		<parent link="red_tool0"/>
 		<child link="palm"/>
-		<origin xyz="0 0 0" rpy="1.57079632679 0 0"/>
+		<origin xyz="0 0 0" rpy="1.57079632679 0 2.35619449019"/>
 	</joint>
 <!-- connecting the red and blue arms together -->
@@ -28,10 +28,10 @@
 		<parent link="ceiling" />
 		<child link="blue_base_link" />
-		<origin xyz="-0.75 0 0" />
+		<origin xyz="-0.715 0.05 0" />
 	</joint>
 	<joint name="ceiling_to_red" type="fixed">
 		<parent link="ceiling" />
 		<child link="red_base_link" />
-		<origin xyz="0.75 0 0" />
+		<origin xyz="0.715 0 0" />
 	</joint>
 	<link name="ceiling" />

File: src/saif_devices/src/dual_arm_description/urdf/red.urdf (robot description, URDF)
Before this commit: robot red, 24 links, 23 joints
Joints:
- joint red_palm_arm: origin xyz=0 0 0 rpy=1.57079632679 0 0 -> xyz=0 0 0 rpy=1.57079632679 0 2.35619449019

File: src/saif_devices/src/dual_arm_description/urdf/red.urdf.xacro (robot description, xacro)
@@ -10,5 +10,5 @@
 		<parent link="red_tool0"/>
 		<child link="palm"/>
-		<origin xyz="0 0 0" rpy="1.57079632679 0 0"/>
+		<origin xyz="0 0 0" rpy="1.57079632679 0 2.35619449019"/>
 	</joint>
 </robot>

Commit message: Added cables to red arm

File: src/saif_devices/src/dual_arm_description/urdf/dual.urdf (robot description, URDF)
Before this commit: robot dual, 61 links, 60 joints
Links:
- added link red_cable_1; visual cylinder length=0.45 radius=0.05
- added link red_cable_2; visual cylinder length=0.45 radius=0.05
- added link red_cable_ee; visual box size=0.1 0.1 0.1
Joints:
- added joint red_2_cable2: type fixed, parent red_upper_arm_link, child red_cable_2, origin xyz=0.0 0.06 0.325
- added joint red_arm_2_cable1: type fixed, parent red_forearm_link, child red_cable_1, origin xyz=0.1 0.0 0.3
- added joint red_arm_2_cable_22: type fixed, parent red_tool0, child red_cable_ee, origin xyz=-0.07 -0.07 -0.03

File: src/saif_devices/src/dual_arm_description/urdf/dual.urdf.xacro (robot description, xacro)
@@ -80,4 +80,43 @@
 		<origin xyz="0 0 0" rpy="1.57079632679 0 2.35619449019"/>
 	</joint>
+	<link name='red_cable_1'>
+		<visual>
+			<geometry>
+				<cylinder length="0.45" radius="0.05"/>
+			</geometry>
+			<material name="black"/>
+		</visual>
+	</link>
+	<joint name='red_arm_2_cable1' type="fixed">
+		<parent link='red_forearm_link'/>
+		<child link='red_cable_1'/>
+		<origin xyz="0.1 0.0 0.3"/>
+	</joint>
+	<link name='red_cable_2'>
+		<visual>
+			<geometry>
+				<cylinder length="0.45" radius="0.05"/>
+			</geometry>
+			<material name="black"/>
+		</visual>
+	</link>
+	<joint name='red_2_cable2' type="fixed">
+		<parent link='red_upper_arm_link'/>
+		<child link='red_cable_2'/>
+		<origin xyz="0.0 0.06 0.325"/>
+	</joint>
+	<link name='red_cable_ee'>
+		<visual>
+			<geometry>
+				<box size="0.1 0.1 0.1"/>
+			</geometry>
+			<material name="black"/>
+		</visual>
+	</link>
+	<joint name='red_arm_2_cable_22' type="fixed">
+		<parent link='red_tool0'/>
+		<child link='red_cable_ee'/>
+		<origin xyz="-0.07 -0.07 -0.03"/>
+	</joint>
 <!-- connecting the red and blue arms together -->
 	<joint name="ceiling_to_blue" type="fixed">

File: src/saif_devices/src/dual_arm_description/urdf/red.urdf (robot description, URDF)
Before this commit: robot red, 24 links, 23 joints
Links:
- added link red_cable_1; visual cylinder length=0.45 radius=0.05
- added link red_cable_2; visual cylinder length=0.45 radius=0.05
- added link red_cable_ee; visual box size=0.1 0.1 0.1
Joints:
- added joint red_2_cable2: type fixed, parent red_upper_arm_link, child red_cable_2, origin xyz=0.0 0.06 0.325
- added joint red_arm_2_cable1: type fixed, parent red_forearm_link, child red_cable_1, origin xyz=0.1 0.0 0.3
- added joint red_arm_2_cable_22: type fixed, parent red_tool0, child red_cable_ee, origin xyz=-0.07 -0.07 -0.03

File: src/saif_devices/src/dual_arm_description/urdf/red.urdf.xacro (robot description, xacro)
@@ -12,3 +12,42 @@
 		<origin xyz="0 0 0" rpy="1.57079632679 0 2.35619449019"/>
 	</joint>
+	<link name='red_cable_1'>
+		<visual>
+			<geometry>
+				<cylinder length="0.45" radius="0.05"/>
+			</geometry>
+			<material name="black"/>
+		</visual>
+	</link>
+	<joint name='red_arm_2_cable1' type="fixed">
+		<parent link='red_forearm_link'/>
+		<child link='red_cable_1'/>
+		<origin xyz="0.1 0.0 0.3"/>
+	</joint>
+	<link name='red_cable_2'>
+		<visual>
+			<geometry>
+				<cylinder length="0.45" radius="0.05"/>
+			</geometry>
+			<material name="black"/>
+		</visual>
+	</link>
+	<joint name='red_2_cable2' type="fixed">
+		<parent link='red_upper_arm_link'/>
+		<child link='red_cable_2'/>
+		<origin xyz="0.0 0.06 0.325"/>
+	</joint>
+	<link name='red_cable_ee'>
+		<visual>
+			<geometry>
+				<box size="0.1 0.1 0.1"/>
+			</geometry>
+			<material name="black"/>
+		</visual>
+	</link>
+	<joint name='red_arm_2_cable_22' type="fixed">
+		<parent link='red_tool0'/>
+		<child link='red_cable_ee'/>
+		<origin xyz="-0.07 -0.07 -0.03"/>
+	</joint>
 </robot>

Commit message: Fixed some urdf issues, presumably due to update, point-based contour following - needs noise filtering.

File: src/saif_devices/src/dual_arm_description/urdf/dual.urdf (robot description, URDF)
Before this commit: robot dual, 64 links, 63 joints
Joints:
- joint red_arm_2_cable_22: origin xyz=-0.07 -0.07 -0.03 -> xyz=0.07 0.0 -0.06
- joint red_palm_arm: origin xyz=0 0 0 rpy=1.57079632679 0 2.35619449019 -> xyz=0 0 0 rpy=1.57079632679 0 -0.78539

File: src/saif_devices/src/dual_arm_description/urdf/dual.urdf.xacro (robot description, xacro)
@@ -78,5 +78,5 @@
 		<parent link="red_tool0"/>
 		<child link="palm"/>
-		<origin xyz="0 0 0" rpy="1.57079632679 0 2.35619449019"/>
+		<origin xyz="0 0 0" rpy="1.57079632679 0 -0.78539"/><!--2.35619449019"/-->
 	</joint>
 	<link name='red_cable_1'>
@@ -117,5 +117,5 @@
 		<parent link='red_tool0'/>
 		<child link='red_cable_ee'/>
-		<origin xyz="-0.07 -0.07 -0.03"/>
+		<origin xyz="0.07 0.0 -0.06"/>
 	</joint>
 <!-- connecting the red and blue arms together -->

File: src/saif_devices/src/dual_arm_description/urdf/red.urdf (robot description, URDF)
Before this commit: robot red, 27 links, 26 joints
Joints:
- joint red_arm_2_cable_22: origin xyz=-0.07 -0.07 -0.03 -> xyz=0.07 0.0 -0.06
- joint red_palm_arm: origin xyz=0 0 0 rpy=1.57079632679 0 2.35619449019 -> xyz=0 0 0 rpy=1.57079632679 0 -0.78539

File: src/saif_devices/src/dual_arm_description/urdf/red.urdf.xacro (robot description, xacro)
@@ -10,5 +10,5 @@
 		<parent link="red_tool0"/>
 		<child link="palm"/>
-		<origin xyz="0 0 0" rpy="1.57079632679 0 2.35619449019"/>
+		<origin xyz="0 0 0" rpy="1.57079632679 0 -0.78539"/>
 	</joint>
 	<link name='red_cable_1'>
@@ -49,5 +49,5 @@
 		<parent link='red_tool0'/>
 		<child link='red_cable_ee'/>
-		<origin xyz="-0.07 -0.07 -0.03"/>
+		<origin xyz="0.07 0.0 -0.06"/>
 	</joint>
 </robot>

Commit message: Better calibrated urdf, contour follower with safer start and end point transitioning.

File: src/saif_devices/src/dual_arm_description/urdf/dual.urdf (robot description, URDF)
Before this commit: robot dual, 64 links, 63 joints
Joints:
- joint ceiling_to_blue: origin xyz=-0.715 0.05 0 -> xyz=-0.745 0.0 -0.04444
- joint ceiling_to_red: origin xyz=0.715 0 0 -> xyz=0.745 0 0

File: src/saif_devices/src/dual_arm_description/urdf/dual.urdf.xacro (robot description, xacro)
@@ -123,10 +123,10 @@
 		<parent link="ceiling" />
 		<child link="blue_base_link" />
-		<origin xyz="-0.715 0.05 0" />
+		<origin xyz="-0.745 0.0 -0.04444" />
 	</joint>
 	<joint name="ceiling_to_red" type="fixed">
 		<parent link="ceiling" />
 		<child link="red_base_link" />
-		<origin xyz="0.715 0 0" />
+		<origin xyz="0.745 0 0" />
 	</joint>
 	<link name="ceiling" />

Commit message: Added force torque sensor to red arm and urdf

File: src/saif_devices/src/dual_arm_description/urdf/dual.urdf (robot description, URDF)
Before this commit: robot dual, 64 links, 63 joints
Links:
- added link red_ft300_mounting_plate; collision mesh filename=package://robotiq_ft_sensor/meshes/collision/mountings/robo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; visual mesh filename=package://robotiq_ft_sensor/meshes/visual/mountings/robotiq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
- added link red_ft300_sensor, mass 0.300; collision mesh filename=package://robotiq_ft_sensor/meshes/collision/robotiq_ft300.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; visual mesh filename=package://robotiq_ft_sensor/meshes/visual/robotiq_ft300.STL
- added link red_robotiq_ft_frame_id
Joints:
- added joint red_ft300_fix: type fixed, parent red_tool0, child red_ft300_mounting_plate, origin xyz=0 0 0 rpy=0 0 0
- added joint red_ft300_mounting_plate: type fixed, parent red_ft300_mounting_plate, child red_ft300_sensor, origin xyz=0 0 0.0415 rpy=0 3.14159265359 0
- added joint red_measurment_joint: type fixed, parent red_ft300_sensor, child red_robotiq_ft_frame_id, origin xyz=0 0 0 rpy=0 3.14159265359 -1.57079632679
- joint red_arm_2_cable_22: origin xyz=0.07 0.0 -0.06 -> xyz=0.00 -0.08 -0.05
- joint red_palm_arm: origin xyz=0 0 0 rpy=1.57079632679 0 -0.78539 -> xyz=0 0 0.05 rpy=1.57079632679 0 0.78539; parent red_tool0 -> red_robotiq_ft_frame_id

File: src/saif_devices/src/dual_arm_description/urdf/dual.urdf.xacro (robot description, xacro)
@@ -72,11 +72,14 @@
 <!-- the red robot -->
 	<xacro:include filename="$(find robotiq_3f_gripper_visualization)/cfg/robotiq-3f-gripper_articulated_macro.xacro" />
+	<xacro:robotiq_ft300 parent="red_tool0" prefix="red_">
+		<origin xyz="0 0 0" rpy="0 0 0"/>
+	</xacro:robotiq_ft300>
 	<!-- arm -->
 	<xacro:ur10_robot prefix="red_" joint_limited="false"/>
 	<xacro:robotiq-3f-gripper_articulated prefix=""/>
 	<joint name="red_palm_arm" type="fixed">
-		<parent link="red_tool0"/>
+		<parent link="red_robotiq_ft_frame_id"/>
 		<child link="palm"/>
-		<origin xyz="0 0 0" rpy="1.57079632679 0 -0.78539"/><!--2.35619449019"/-->
+		<origin xyz="0 0 0.05" rpy="1.57079632679 0 0.78539"/><!--2.35619449019"/-->
 	</joint>
 	<link name='red_cable_1'>
@@ -117,5 +120,5 @@
 		<parent link='red_tool0'/>
 		<child link='red_cable_ee'/>
-		<origin xyz="0.07 0.0 -0.06"/>
+		<origin xyz="0.00 -0.08 -0.05"/>
 	</joint>
 <!-- connecting the red and blue arms together -->

File: src/saif_devices/src/dual_arm_description/urdf/red.urdf (robot description, URDF)
Before this commit: robot red, 27 links, 26 joints
Links:
- added link red_ft300_mounting_plate; collision mesh filename=package://robotiq_ft_sensor/meshes/collision/mountings/robo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; visual mesh filename=package://robotiq_ft_sensor/meshes/visual/mountings/robotiq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
- added link red_ft300_sensor, mass 0.300; collision mesh filename=package://robotiq_ft_sensor/meshes/collision/robotiq_ft300.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; visual mesh filename=package://robotiq_ft_sensor/meshes/visual/robotiq_ft300.STL
- added link red_robotiq_ft_frame_id
Joints:
- added joint red_ft300_fix: type fixed, parent red_tool0, child red_ft300_mounting_plate, origin xyz=0 0 0 rpy=0 0 0
- added joint red_ft300_mounting_plate: type fixed, parent red_ft300_mounting_plate, child red_ft300_sensor, origin xyz=0 0 0.0415 rpy=0 3.14159265359 0
- added joint red_measurment_joint: type fixed, parent red_ft300_sensor, child red_robotiq_ft_frame_id, origin xyz=0 0 0 rpy=0 3.14159265359 -1.57079632679
- joint red_arm_2_cable_22: origin xyz=0.07 0.0 -0.06 -> xyz=0.00 -0.08 -0.05
- joint red_palm_arm: origin xyz=0 0 0 rpy=1.57079632679 0 -0.78539 -> xyz=0 0 0.05 rpy=1.57079632679 0 0.78539; parent red_tool0 -> red_robotiq_ft_frame_id

File: src/saif_devices/src/dual_arm_description/urdf/red.urdf.xacro (robot description, xacro)
@@ -4,11 +4,15 @@
 	<xacro:include filename="$(find ur_description)/urdf/common.gazebo.xacro" />
 	<xacro:include filename="$(find ur_description)/urdf/ur10.urdf.xacro" />
+        <xacro:include filename="$(find robotiq_ft_sensor)/urdf/robotiq_ft300.urdf.xacro"/>
 	<!-- arm -->
 	<xacro:ur10_robot prefix="red_" joint_limited="false"/>
 	<xacro:robotiq-3f-gripper_articulated prefix=""/>
+        <xacro:robotiq_ft300 parent="red_tool0" prefix="red_">
+                <origin xyz="0 0 0" rpy="0 0 0"/>
+        </xacro:robotiq_ft300>
 	<joint name="red_palm_arm" type="fixed">
-		<parent link="red_tool0"/>
+		<parent link="red_robotiq_ft_frame_id"/>
 		<child link="palm"/>
-		<origin xyz="0 0 0" rpy="1.57079632679 0 -0.78539"/>
+		<origin xyz="0 0 0.05" rpy="1.57079632679 0 0.78539"/>
 	</joint>
 	<link name='red_cable_1'>
@@ -49,5 +53,5 @@
 		<parent link='red_tool0'/>
 		<child link='red_cable_ee'/>
-		<origin xyz="0.07 0.0 -0.06"/>
+		<origin xyz="0.00 -0.08 -0.05"/>
 	</joint>
 </robot>
