Commit message: Changed ft sensor tf tree

File: src/saif_devices/src/dual_arm_description/urdf/dual.urdf.xacro (robot description, xacro)
@@ -7,10 +7,10 @@
 	<xacro:include filename="$(find robotiq_ft_sensor)/urdf/robotiq_ft300.urdf.xacro"/>
 	<xacro:robotiq_ft300 parent="blue_tool0" prefix="blue_">
-		<origin xyz="0 0 0" rpy="0 0 0"/>
+		<origin xyz="0 0 0" rpy="0 0 -1.57079632679"/>
 	</xacro:robotiq_ft300>
 	<!-- arm -->
 	<xacro:ur10_robot prefix="blue_" joint_limited="false"/>
  	<xacro:robotiq_85_gripper prefix="" parent="blue_robotiq_ft_frame_id">
-		 <origin xyz="0.0 0.0 0.0" rpy="0 -1.57079632679 0"/>
+		 <origin xyz="0.0 0.0 0.0" rpy="0 -1.57079632679 1.57079632679"/>
 	</xacro:robotiq_85_gripper>
 <link name='cable_1'>
@@ -73,5 +73,5 @@
 	<xacro:include filename="$(find robotiq_3f_gripper_visualization)/cfg/robotiq-3f-gripper_articulated_macro.xacro" />
 	<xacro:robotiq_ft300 parent="red_tool0" prefix="red_">
-		<origin xyz="0 0 0" rpy="0 0 0"/>
+		<origin xyz="0 0 0" rpy="0 0 -1.57079632679"/>
 	</xacro:robotiq_ft300>
 	<!-- arm -->
@@ -81,5 +81,5 @@
 		<parent link="red_robotiq_ft_frame_id"/>
 		<child link="palm"/>
-		<origin xyz="0 0 0.05" rpy="1.57079632679 0 0.78539"/><!--2.35619449019"/-->
+		<origin xyz="0 0 0.05" rpy="1.57079632679 0 2.35619449019"/><!--2.35619449019"/-->
 	</joint>
 	<link name='red_cable_1'>
