Commit message: Added cabling and real sense sensor to blue urdf

File: src/saif_devices/src/dual_arm_description/urdf/blue.urdf (robot description, URDF)
Before this commit: robot blue, 22 links, 21 joints
Links:
- added link cable_1; visual cylinder length=0.45 radius=0.05
- added link cable_2; visual cylinder length=0.45 radius=0.05
- added link cable_ee; visual box size=0.1 0.1 0.1
- added link camera_bottom_screw_frame
- added link camera_color_frame
- added link camera_color_optical_frame
- added link camera_depth_frame
- added link camera_depth_optical_frame
- added link camera_left_ir_frame
- added link camera_left_ir_optical_frame
- added link camera_link, mass 0.564; collision box size=0.02505 0.09 0.025; visual mesh filename=package://dual_arm_description/meshes/d435.dae
- added link camera_right_ir_frame
- added link camera_right_ir_optical_frame
- added link realsense_mount; visual box size=0.05 0.05 0.05
Joints:
- added joint arm_2_cable1: type fixed, parent blue_forearm_link, child cable_1, origin xyz=0.1 0.0 0.3
- added joint arm_2_cable2: type fixed, parent blue_upper_arm_link, child cable_2, origin xyz=0.0 0.06 0.325
- added joint arm_2_cable_22: type fixed, parent blue_tool0, child cable_ee, origin xyz=-0.1 0.0 0.06
- added joint camera_color_joint: type fixed, parent camera_depth_frame, child camera_color_frame, origin xyz=0 0.015 0 rpy=0 0 0
- added joint camera_color_optical_joint: type fixed, parent camera_color_frame, child camera_color_optical_frame, origin xyz=0 0 0 rpy=-1.57079632679 0 -1.57079632679
- added joint camera_depth_joint: type fixed, parent camera_link, child camera_depth_frame, origin xyz=0 0 0 rpy=0 0 0
- added joint camera_depth_optical_joint: type fixed, parent camera_depth_frame, child camera_depth_optical_frame, origin xyz=0 0 0 rpy=-1.57079632679 0 -1.57079632679
- added joint camera_joint: type fixed, parent gripper_base_link, child camera_bottom_screw_frame, origin xyz=0.02 0 -0.1 rpy=0 0 3.14159
- added joint camera_left_ir_joint: type fixed, parent camera_depth_frame, child camera_left_ir_frame, origin xyz=0 0.0 0 rpy=0 0 0
- added joint camera_left_ir_optical_joint: type fixed, parent camera_left_ir_frame, child camera_left_ir_optical_frame, origin xyz=0 0 0 rpy=-1.57079632679 0 -1.57079632679
- added joint camera_link_joint: type fixed, parent camera_bottom_screw_frame, child camera_link, origin xyz=0 0.0175 0.0125 rpy=0 0 0
- added joint camera_right_ir_joint: type fixed, parent camera_depth_frame, child camera_right_ir_frame, origin xyz=0 -0.05 0 rpy=0 0 0
- added joint camera_right_ir_optical_joint: type fixed, parent camera_right_ir_frame, child camera_right_ir_optical_frame, origin xyz=0 0 0 rpy=-1.57079632679 0 -1.57079632679
- added joint ee_2_realsense_22: type fixed, parent gripper_base_link, child realsense_mount, origin xyz=0.02 0.0 -0.05

File: src/saif_devices/src/dual_arm_description/urdf/blue.urdf.xacro (robot description, xacro)
@@ -8,4 +8,57 @@
 		<origin xyz="0 0 0" rpy="0 0 0"/>
 	</xacro:robotiq_ft300>
+	<link name='cable_1'>
+		<visual>
+			<geometry>
+				<cylinder length="0.45" radius="0.05"/>
+			</geometry>
+			<material name="black"/>
+		</visual>
+	</link>
+	<joint name='arm_2_cable1' type="fixed">
+		<parent link='blue_forearm_link'/>
+		<child link='cable_1'/>
+		<origin xyz="0.1 0.0 0.3"/>
+	</joint>
+	<link name='cable_2'>
+		<visual>
+			<geometry>
+				<cylinder length="0.45" radius="0.05"/>
+			</geometry>
+			<material name="black"/>
+		</visual>
+	</link>
+	<joint name='arm_2_cable2' type="fixed">
+		<parent link='blue_upper_arm_link'/>
+		<child link='cable_2'/>
+		<origin xyz="0.0 0.06 0.325"/>
+	</joint>
+	<link name='cable_ee'>
+		<visual>
+			<geometry>
+				<box size="0.1 0.1 0.1"/>
+			</geometry>
+			<material name="black"/>
+		</visual>
+	</link>
+	<joint name='arm_2_cable_22' type="fixed">
+		<parent link='blue_tool0'/>
+		<child link='cable_ee'/>
+		<origin xyz="-0.1 0.0 0.06"/>
+	</joint>
+	<link name='realsense_mount'>
+		<visual>
+			<geometry>
+				<box size="0.05 0.05 0.05"/>
+			</geometry>
+			<material name="black"/>
+		</visual>
+	</link>
+	<joint name='ee_2_realsense_22' type="fixed">
+		<parent link='gripper_base_link'/>
+		<child link='realsense_mount'/>
+		<origin xyz="0.02 0.0 -0.05"/>
+	</joint>
+	<xacro:include filename="$(find dual_arm_description)/urdf/d435.urdf.xacro"/>
 	<!-- arm -->
 	<xacro:ur10_robot prefix="blue_" joint_limited="false"/>
@@ -13,3 +66,6 @@
 		 <origin xyz="0.0 0.0 0.0" rpy="0 -1.57079632679 0"/>
 	</xacro:robotiq_85_gripper>
+	<xacro:sensor_d435 parent="gripper_base_link">
+		<origin xyz ="0.02 0 -0.1" rpy="0 0 3.14159"/>
+	</xacro:sensor_d435>
 </robot>

File: src/saif_devices/src/dual_arm_description/urdf/dual.urdf (robot description, URDF)
Before this commit: robot dual, 47 links, 46 joints
Links:
- added link cable_1; visual cylinder length=0.45 radius=0.05
- added link cable_2; visual cylinder length=0.45 radius=0.05
- added link cable_ee; visual box size=0.1 0.1 0.1
- added link camera_bottom_screw_frame
- added link camera_color_frame
- added link camera_color_optical_frame
- added link camera_depth_frame
- added link camera_depth_optical_frame
- added link camera_left_ir_frame
- added link camera_left_ir_optical_frame
- added link camera_link, mass 0.564; collision box size=0.02505 0.09 0.025; visual mesh filename=package://dual_arm_description/meshes/d435.dae
- added link camera_right_ir_frame
- added link camera_right_ir_optical_frame
- added link realsense_mount; visual box size=0.05 0.05 0.05
Joints:
- added joint arm_2_cable1: type fixed, parent blue_forearm_link, child cable_1, origin xyz=0.1 0.0 0.3
- added joint arm_2_cable2: type fixed, parent blue_upper_arm_link, child cable_2, origin xyz=0.0 0.06 0.325
- added joint arm_2_cable_22: type fixed, parent blue_tool0, child cable_ee, origin xyz=-0.1 0.0 0.06
- added joint camera_color_joint: type fixed, parent camera_depth_frame, child camera_color_frame, origin xyz=0 0.015 0 rpy=0 0 0
- added joint camera_color_optical_joint: type fixed, parent camera_color_frame, child camera_color_optical_frame, origin xyz=0 0 0 rpy=-1.57079632679 0 -1.57079632679
- added joint camera_depth_joint: type fixed, parent camera_link, child camera_depth_frame, origin xyz=0 0 0 rpy=0 0 0
- added joint camera_depth_optical_joint: type fixed, parent camera_depth_frame, child camera_depth_optical_frame, origin xyz=0 0 0 rpy=-1.57079632679 0 -1.57079632679
- added joint camera_joint: type fixed, parent gripper_base_link, child camera_bottom_screw_frame, origin xyz=0.02 0 -0.1 rpy=0 0 3.14159
- added joint camera_left_ir_joint: type fixed, parent camera_depth_frame, child camera_left_ir_frame, origin xyz=0 0.0 0 rpy=0 0 0
- added joint camera_left_ir_optical_joint: type fixed, parent camera_left_ir_frame, child camera_left_ir_optical_frame, origin xyz=0 0 0 rpy=-1.57079632679 0 -1.57079632679
- added joint camera_link_joint: type fixed, parent camera_bottom_screw_frame, child camera_link, origin xyz=0 0.0175 0.0125 rpy=0 0 0
- added joint camera_right_ir_joint: type fixed, parent camera_depth_frame, child camera_right_ir_frame, origin xyz=0 -0.05 0 rpy=0 0 0
- added joint camera_right_ir_optical_joint: type fixed, parent camera_right_ir_frame, child camera_right_ir_optical_frame, origin xyz=0 0 0 rpy=-1.57079632679 0 -1.57079632679
- added joint ee_2_realsense_22: type fixed, parent gripper_base_link, child realsense_mount, origin xyz=0.02 0.0 -0.05

File: src/saif_devices/src/dual_arm_description/urdf/dual.urdf.xacro (robot description, xacro)
@@ -14,4 +14,60 @@
 		 <origin xyz="0.0 0.0 0.0" rpy="0 -1.57079632679 0"/>
 	</xacro:robotiq_85_gripper>
+<link name='cable_1'>
+		<visual>
+			<geometry>
+				<cylinder length="0.45" radius="0.05"/>
+			</geometry>
+			<material name="black"/>
+		</visual>
+	</link>
+	<joint name='arm_2_cable1' type="fixed">
+		<parent link='blue_forearm_link'/>
+		<child link='cable_1'/>
+		<origin xyz="0.1 0.0 0.3"/>
+	</joint>
+	<link name='cable_2'>
+		<visual>
+			<geometry>
+				<cylinder length="0.45" radius="0.05"/>
+			</geometry>
+			<material name="black"/>
+		</visual>
+	</link>
+	<joint name='arm_2_cable2' type="fixed">
+		<parent link='blue_upper_arm_link'/>
+		<child link='cable_2'/>
+		<origin xyz="0.0 0.06 0.325"/>
+	</joint>
+	<link name='cable_ee'>
+		<visual>
+			<geometry>
+				<box size="0.1 0.1 0.1"/>
+			</geometry>
+			<material name="black"/>
+		</visual>
+	</link>
+	<joint name='arm_2_cable_22' type="fixed">
+		<parent link='blue_tool0'/>
+		<child link='cable_ee'/>
+		<origin xyz="-0.1 0.0 0.06"/>
+	</joint>
+	<link name='realsense_mount'>
+		<visual>
+			<geometry>
+				<box size="0.05 0.05 0.05"/>
+			</geometry>
+			<material name="black"/>
+		</visual>
+	</link>
+	<joint name='ee_2_realsense_22' type="fixed">
+		<parent link='gripper_base_link'/>
+		<child link='realsense_mount'/>
+		<origin xyz="0.02 0.0 -0.05"/>
+	</joint>
+	<xacro:include filename="$(find dual_arm_description)/urdf/d435.urdf.xacro"/>
+	<xacro:sensor_d435 parent="gripper_base_link">
+		<origin xyz ="0.02 0 -0.1" rpy="0 0 3.14159"/>
+	</xacro:sensor_d435>
 <!-- the red robot -->
 	<xacro:include filename="$(find robotiq_3f_gripper_visualization)/cfg/robotiq-3f-gripper_articulated_macro.xacro" />

Commit message: Some contour debugging - normals issues

File: src/saif_devices/src/dual_arm_description/urdf/blue.urdf (robot description, URDF)
Before this commit: robot blue, 36 links, 35 joints
Joints:
- joint camera_joint: origin xyz=0.02 0 -0.1 rpy=0 0 3.14159 -> xyz=0.02 0 -0.1 rpy=0 3.14159 3.14159

File: src/saif_devices/src/dual_arm_description/urdf/blue.urdf.xacro (robot description, xacro)
@@ -67,5 +67,5 @@
 	</xacro:robotiq_85_gripper>
 	<xacro:sensor_d435 parent="gripper_base_link">
-		<origin xyz ="0.02 0 -0.1" rpy="0 0 3.14159"/>
+		<origin xyz ="0.02 0 -0.1" rpy="0 3.14159 3.14159"/>
 	</xacro:sensor_d435>
 </robot>

File: src/saif_devices/src/dual_arm_description/urdf/dual.urdf (robot description, URDF)
Before this commit: robot dual, 64 links, 63 joints
Joints:
- joint camera_joint: origin xyz=0.02 0 -0.1 rpy=0 0 3.14159 -> xyz=0.02 0 -0.1 rpy=0 3.14159 3.14159

File: src/saif_devices/src/dual_arm_description/urdf/dual.urdf.xacro (robot description, xacro)
@@ -68,5 +68,5 @@
 	<xacro:include filename="$(find dual_arm_description)/urdf/d435.urdf.xacro"/>
 	<xacro:sensor_d435 parent="gripper_base_link">
-		<origin xyz ="0.02 0 -0.1" rpy="0 0 3.14159"/>
+		<origin xyz ="0.02 0 -0.1" rpy="0 3.14159 3.14159"/>
 	</xacro:sensor_d435>
 <!-- the red robot -->

Commit message: Updated all urdfs with correct ft rotation

File: src/saif_devices/src/dual_arm_description/urdf/blue.urdf (robot description, URDF)
Before this commit: robot blue, 36 links, 35 joints
Joints:
- joint blue_ft300_fix: origin xyz=0 0 0 rpy=0 0 0 -> xyz=0 0 0 rpy=0 0 -1.57079632679
- joint gripper_base_joint: origin xyz=0.0 0.0 0.0 rpy=0 -1.57079632679 0 -> xyz=0.0 0.0 0.0 rpy=0 -1.57079632679 1.57079632679

File: src/saif_devices/src/dual_arm_description/urdf/blue.urdf.xacro (robot description, xacro)
@@ -6,5 +6,5 @@
 	<xacro:include filename="$(find robotiq_ft_sensor)/urdf/robotiq_ft300.urdf.xacro"/>
 	<xacro:robotiq_ft300 parent="blue_tool0" prefix="blue_">
-		<origin xyz="0 0 0" rpy="0 0 0"/>
+		<origin xyz="0 0 0" rpy="0 0 -1.57079632679"/>
 	</xacro:robotiq_ft300>
 	<link name='cable_1'>
@@ -64,5 +64,5 @@
 	<xacro:ur10_robot prefix="blue_" joint_limited="false"/>
  	<xacro:robotiq_85_gripper prefix="" parent="blue_robotiq_ft_frame_id">
-		 <origin xyz="0.0 0.0 0.0" rpy="0 -1.57079632679 0"/>
+		 <origin xyz="0.0 0.0 0.0" rpy="0 -1.57079632679 1.57079632679"/>
 	</xacro:robotiq_85_gripper>
 	<xacro:sensor_d435 parent="gripper_base_link">

File: src/saif_devices/src/dual_arm_description/urdf/dual.urdf (robot description, URDF)
Before this commit: robot dual, 67 links, 66 joints
Joints:
- joint blue_ft300_fix: origin xyz=0 0 0 rpy=0 0 0 -> xyz=0 0 0 rpy=0 0 -1.57079632679
- joint gripper_base_joint: origin xyz=0.0 0.0 0.0 rpy=0 -1.57079632679 0 -> xyz=0.0 0.0 0.0 rpy=0 -1.57079632679 1.57079632679
- joint red_ft300_fix: origin xyz=0 0 0 rpy=0 0 0 -> xyz=0 0 0 rpy=0 0 -1.57079632679
- joint red_palm_arm: origin xyz=0 0 0.05 rpy=1.57079632679 0 0.78539 -> xyz=0 0 0.05 rpy=1.57079632679 0 2.35619449019

File: src/saif_devices/src/dual_arm_description/urdf/red.urdf (robot description, URDF)
Before this commit: robot red, 30 links, 29 joints
Joints:
- joint red_ft300_fix: origin xyz=0 0 0 rpy=0 0 0 -> xyz=0 0 0 rpy=0 0 -1.57079632679
- joint red_palm_arm: origin xyz=0 0 0.05 rpy=1.57079632679 0 0.78539 -> xyz=0 0 0.05 rpy=1.57079632679 0 2.35619449019

File: src/saif_devices/src/dual_arm_description/urdf/red.urdf.xacro (robot description, xacro)
@@ -8,11 +8,11 @@
 	<xacro:ur10_robot prefix="red_" joint_limited="false"/>
 	<xacro:robotiq-3f-gripper_articulated prefix=""/>
-        <xacro:robotiq_ft300 parent="red_tool0" prefix="red_">
-                <origin xyz="0 0 0" rpy="0 0 0"/>
-        </xacro:robotiq_ft300>
+	<xacro:robotiq_ft300 parent="red_tool0" prefix="red_">
+		<origin xyz="0 0 0" rpy="0 0 -1.57079632679"/>
+	</xacro:robotiq_ft300>
 	<joint name="red_palm_arm" type="fixed">
 		<parent link="red_robotiq_ft_frame_id"/>
 		<child link="palm"/>
-		<origin xyz="0 0 0.05" rpy="1.57079632679 0 0.78539"/>
+		<origin xyz="0 0 0.05" rpy="1.57079632679 0 2.35619449019"/><!--2.35619449019"/-->
 	</joint>
 	<link name='red_cable_1'>
